File: USB2TTL.kicad_pcb (KiCad board)
At the start: 2 copper layers, 30 x 20 mm, 30 parts, among them J1 USB_A, J2 Conn_01x05, Q1 SiA517DJ, SW1 TS-1187A-B-A-B, SW2 TS-1187A-B-A-B, U1 SPX3819M5-L-3-3, U2 CH343P

Commit message: Done V1.0
Parts:
- J2: footprint Connector_PinHeader_2.54mm:PinHeader_1x05_P2.54mm_Horizontal -> JLC-SMT:PinHeader_1x05_P2.54mm_Horizontal_SMD
- moved J2 1.56 mm to (127.5, 104.9)
Routing:
- net /TXD: track 25.5 -> 20.6 mm, vias 1 -> 2
- net /BOOT: track 28.9 -> 24.0 mm, vias 2 -> 3
- net /RXD: track 27.1 -> 22.2 mm, vias 1 -> 2
- net /VOUT: track 9.20 -> 8.52 mm
- net GND: vias 66 -> 78
Other:
- outline, holes or cut-outs redrawn
- board text added: "5V"
- board text added: "B0"
- board text added: "CH343P"
- board text added: "DTR"
- board text added: "RTS"
- board text added: "RX"
- board text added: "TX"
- board text added: "USB SERIAL V1.0"
- board text added: "XiNGRZ"
